File: pcb_puissance/connectors.kicad_sch (KiCad schematic)
At the start: 34 parts, among them J10 1755736, J11 USB_C_Receptacle_USB2.0_16P, J12 1755736, J13 1755736, J14 Conn_02x06_Odd_Even, J15 1755736, J16 1755736, J17 Conn_02x06_Odd_Even, J18 1755736, J19 1755736, J20 Conn_02x06_Odd_Even, J21 1755736, J22 1755736, Q7 STL40DN3LLH5, U3 INA236BIDDFR, U4 INA236AIDDFR, U5 INA236AIDDFR, U6 INA236AIDDFR, U9 TCPP02-M18

Commit message: dernieres retouches suite changement de repo
Parts:
- U3, U4, U5, U6: footprint SOT23-8_DDF_TEX -> Modelec:SOT23-8_DDF_TEX
Changed lines of the file:
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@@
 	(title_block
 		(title "Power output connectors")
-		(date "2025-02-10")
-		(rev "3")
+		(date "2025-03-06")
+		(rev "4")
 		(company "Modelec")
 		(comment 2 "USBC-Power Delivery 5V15 capacity, programmable from the STM32 via I2C")
@@
 	)
 	(bus_entry
+		(at 114.3 179.07)
+		(size 2.54 2.54)
+		(stroke
+			(width 0)
+			(type default)
+		)
+	)
+	(bus_entry
 		(at 85.09 138.43)
 		(size -2.54 2.54)
@@
 	)
 	(bus_entry
+		(at 111.76 179.07)
+		(size 2.54 2.54)
+		(stroke
+			(width 0)
+			(type default)
+		)
+	)
+	(bus_entry
 		(at 227.33 17.78)
 		(size 2.54 -2.54)
@@
 	(wire
 		(pts
+			(xy 111.76 168.91) (xy 111.76 179.07)
+		)
+		(stroke
+			(width 0)
+			(type default)
+		)
+	)
+	(wire
+		(pts
 			(xy 129.54 68.58) (xy 134.62 68.58)
 		)
@@
 	(wire
 		(pts
+			(xy 114.3 168.91) (xy 114.3 179.07)
+		)
+		(stroke
+			(width 0)
+			(type default)
+		)
+	)
+	(wire
+		(pts
 			(xy 50.8 137.16) (xy 50.8 135.89)
 		)
@@
 		)
 	)
+	(bus
+		(pts
+			(xy 116.84 181.61) (xy 121.92 181.61)
+		)
+		(stroke
+			(width 0)
+			(type default)
+		)
+	)
 	(wire
 		(pts
@@
 		)
 	)
+	(bus
+		(pts
+			(xy 116.84 181.61) (xy 114.3 181.61)
+		)
+		(stroke
+			(width 0)
+			(type default)
+		)
+	)
 	(wire
 		(pts
@@
 		)
 	)
+	(label "SCL"
+		(at 111.76 179.07 90)
+		(effects
+			(font
+				(size 1.27 1.27)
+			)
+			(justify left bottom)
+		)
+	)
 	(label "CC1"
 		(at 85.09 146.05 0)
@@
 		)
 	)
+	(label "SDA"
+		(at 114.3 179.07 90)
+		(effects
+			(font
+				(size 1.27 1.27)
+			)
+			(justify left bottom)
+		)
+	)
 	(label "SCL"
 		(at 50.8 19.05 270)
@@
 		)
 	)
-	(hierarchical_label "SDA"
-		(shape bidirectional)
-		(at 114.3 168.91 270)
-		(effects
-			(font
-				(size 1.27 1.27)
-			)
-			(justify right)
-		)
-	)
 	(hierarchical_label "3V3"
 		(shape input)
@@
 		)
 	)
-	(hierarchical_label "SCL"
-		(shape bidirectional)
-		(at 111.76 168.91 270)
+	(hierarchical_label "3V3"
+		(shape input)
+		(at 72.39 142.24 270)
 		(effects
 			(font
@@
 		)
 	)
-	(hierarchical_label "3V3"
-		(shape input)
-		(at 72.39 142.24 270)
+	(hierarchical_label "{I2C}"
+		(shape bidirectional)
+		(at 121.92 181.61 0)
 		(effects
 			(font
 				(size 1.27 1.27)
 			)
-			(justify right)
+			(justify left)
 		)
 	)
@@
 			)
 		)
-		(property "Footprint" "SOT23-8_DDF_TEX"
+		(property "Footprint" "Modelec:SOT23-8_DDF_TEX"
 			(at 134.62 58.42 0)
 			(effects
@@
 					(size 1.27 1.27)
 				)
+				(hide yes)
 			)
 		)
@@
 					(size 1.27 1.27)
 				)
+				(hide yes)
 			)
 		)
@@
 					(size 1.27 1.27)
 				)
+				(hide yes)
 			)
 		)
@@
 					(size 1.27 1.27)
 				)
+				(hide yes)
 			)
 		)
@@
 					(size 1.27 1.27)
 				)
+				(hide yes)
 			)
 		)
@@
 			)
 		)
-		(property "Footprint" "SOT23-8_DDF_TEX"
+		(property "Footprint" "Modelec:SOT23-8_DDF_TEX"
 			(at 43.18 58.42 0)
 			(effects
@@
 					(size 1.27 1.27)
 				)
+				(hide yes)
 			)
 		)
@@
 		(on_board yes)
 		(dnp no)
-		(fields_autoplaced yes)
 		(property "Reference" "C21"
 			(at 142.24 129.5399 0)
@@
 		)
 		(property "Manufacturer_Part_Number" "VJ0805Y104KXAMR"
-			(at 138.43 130.81 0)
+			(at 138.43 131.826 0)
 			(effects
 				(font
 					(size 1.27 1.27)
 				)
+				(hide yes)
 			)
 		)
@@
 			)
 		)
-		(property "Footprint" "SOT23-8_DDF_TEX"
+		(property "Footprint" "Modelec:SOT23-8_DDF_TEX"
 			(at 219.71 57.15 0)
 			(effects
@@
 					(size 1.27 1.27)
 				)
+				(hide yes)
 			)
 		)
@@
 		(on_board yes)
 		(dnp no)
-		(fields_autoplaced yes)
 		(property "Reference" "D4"
 			(at 154.94 101.9176 90)
@@
 		)
 		(property "Manufacturer_Part_Number" "ESDA25P35-1U1M"
-			(at 157.48 100.33 0)
+			(at 166.37 97.028 90)
 			(effects
 				(font
 					(size 1.27 1.27)
 				)
+				(hide yes)
 			)
 		)
@@
 					(size 1.27 1.27)
 				)
+				(hide yes)
 			)
 		)
@@
 		)
 		(property "Manufacturer_Part_Number" "VJ0805G225KXQTW1BC"
-			(at 176.53 100.33 0)
+			(at 188.468 97.028 0)
 			(effects
 				(font
 					(size 1.27 1.27)
 				)
+				(hide yes)
 			)
 		)
@@
 			)
 		)
-		(property "Footprint" "SOT23-8_DDF_TEX"
+		(property "Footprint" "Modelec:SOT23-8_DDF_TEX"
 			(at 45.72 132.08 0)
 			(effects
@@
 					(size 1.27 1.27)
 				)
+				(hide yes)
 			)
 		)
@@
 		(on_board yes)
 		(dnp no)
-		(fields_autoplaced yes)
 		(property "Reference" "C19"
 			(at 154.94 148.5899 0)
@@
 		)
 		(property "Manufacturer_Part_Number" "VJ0805A331FXACW1BC"
-			(at 151.13 149.86 0)
+			(at 151.13 152.146 0)
 			(effects
 				(font
 					(size 1.27 1.27)
 				)
+				(hide yes)
 			)
 		)
@@
 					(size 1.27 1.27)
 				)
+				(hide yes)
 			)
 		)
