File: pcb_puissance/converters.kicad_sch (KiCad schematic)
At the start: 25 parts, among them Q10 NMOS, Q11 NMOS, Q9 NMOS

Commit message: dernieres retouches suite changement de repo
Parts:
- PS2, PS3, PS5: footprint THN301211 -> Modelec:THN301211
- PS4: footprint TEN_50-2411 -> Modelec:TEN_50-2411
Other:
- company: (none) -> Modelec
- title: (none) -> Power converters
Changed lines of the file:
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@@
 	(paper "A4")
 	(title_block
-		(date "2025-02-10")
+		(title "Power converters")
+		(date "2025-03-06")
+		(rev "4")
+		(company "Modelec")
+		(comment 1 "Disable software emergency stop bridging the 3 jumpers")
+		(comment 2 "Power converters and control via physical and stm32 software emergency stop")
 	)
 	(text "24V 1,25A Power Supply\n"
@@
 		)
 		(property "Manufacturer_Part_Number" "2N7002-7-F"
-			(at 86.36 167.64 0)
+			(at 97.028 171.196 0)
 			(effects
 				(font
@@
 					(size 1.27 1.27)
 				)
+				(hide yes)
 			)
 		)
@@
 		)
 		(property "Manufacturer_Part_Number" "2N7002-7-F"
-			(at 88.9 81.28 0)
+			(at 99.568 84.836 0)
 			(effects
 				(font
@@
 			)
 		)
-		(property "Footprint" "THN301211"
+		(property "Footprint" "Modelec:THN301211"
 			(at 185.42 160.96 0)
 			(effects
@@
 		(on_board yes)
 		(dnp no)
-		(fields_autoplaced yes)
 		(property "Reference" "D7"
 			(at 95.1865 143.51 0)
@@
 		)
 		(property "Manufacturer_Part_Number" "BAS70-06"
-			(at 95.25 152.4 0)
+			(at 102.616 154.686 0)
 			(effects
 				(font
@@
 					(size 1.27 1.27)
 				)
+				(hide yes)
 			)
 		)
@@
 			)
 		)
-		(property "Footprint" "TEN_50-2411"
+		(property "Footprint" "Modelec:TEN_50-2411"
 			(at 182.88 204.14 0)
 			(effects
@@
 					(size 1.27 1.27)
 				)
+				(hide yes)
 			)
 		)
@@
 					(size 1.27 1.27)
 				)
+				(hide yes)
 			)
 		)
@@
 			)
 		)
-		(property "Footprint" "THN301211"
+		(property "Footprint" "Modelec:THN301211"
 			(at 185.42 247.32 0)
 			(effects
@@
 					(size 1.27 1.27)
 				)
+				(hide yes)
 			)
 		)
@@
 					(size 1.27 1.27)
 				)
+				(hide yes)
 			)
 		)
@@
 		)
 		(property "Manufacturer_Part_Number" "2N7002-7-F"
-			(at 87.63 124.46 0)
+			(at 98.806 128.016 0)
 			(effects
 				(font
@@
 					(size 1.27 1.27)
 				)
+				(hide yes)
 			)
 		)
@@
 		(on_board yes)
 		(dnp no)
-		(fields_autoplaced yes)
 		(property "Reference" "D6"
 			(at 95.1865 100.33 0)
@@
 		)
 		(property "Manufacturer_Part_Number" "BAS70-06"
-			(at 95.25 109.22 0)
+			(at 102.87 111.506 0)
 			(effects
 				(font
@@
 					(size 1.27 1.27)
 				)
+				(hide yes)
 			)
 		)
@@
 		)
 		(property "Manufacturer_Part_Number" "BAS70-06"
-			(at 96.52 66.04 0)
+			(at 103.124 67.818 0)
 			(effects
 				(font
@@
 			)
 		)
-		(property "Footprint" "THN301211"
+		(property "Footprint" "Modelec:THN301211"
 			(at 185.42 124.13 0)
 			(effects
