File: pcb_puissance/microcontroller.kicad_sch (KiCad schematic)
At the start: 25 parts, among them J7 Conn_02x10_Odd_Even, J8 Conn_ST_STDC14, Q8 NPN, U10 MCP9808T-E/MS, U2 STM32G491KEU6

Commit message: dernieres retouches suite changement de repo
Parts:
- U10: footprint MSOP8_MC_MCH -> Modelec:MSOP8_MC_MCH
Connections:
- net 3V3: now also J8.3 (VCC)
Changed lines of the file:
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@@
 	(title_block
 		(title "Power supply controller")
-		(date "2025-02-10")
-		(rev "3")
+		(date "2025-03-06")
+		(rev "4")
 		(company "Modelec")
 		(comment 1 "read temperature, power measurements and validity status of the inputs")
@@
 	(wire
 		(pts
-			(xy 99.06 160.02) (xy 101.6 160.02)
-		)
-		(stroke
-			(width 0)
-			(type default)
-		)
-	)
-	(wire
-		(pts
 			(xy 128.27 140.97) (xy 140.97 140.97)
 		)
@@
 	(wire
 		(pts
+			(xy 46.99 54.61) (xy 46.99 59.69)
+		)
+		(stroke
+			(width 0)
+			(type default)
+		)
+	)
+	(wire
+		(pts
 			(xy 132.08 27.94) (xy 132.08 34.29)
 		)
@@
 	(hierarchical_label "3V3"
 		(shape input)
+		(at 46.99 54.61 180)
+		(effects
+			(font
+				(size 1.27 1.27)
+			)
+			(justify right)
+		)
+	)
+	(hierarchical_label "3V3"
+		(shape input)
 		(at 224.79 26.67 90)
 		(effects
@@
 					(size 1.27 1.27)
 				)
+				(hide yes)
 			)
 		)
@@
 					(size 1.27 1.27)
 				)
+				(hide yes)
 			)
 		)
@@
 					(size 1.27 1.27)
 				)
+				(hide yes)
 			)
 		)
@@
 					(size 1.27 1.27)
 				)
+				(hide yes)
 			)
 		)
@@
 					(size 1.27 1.27)
 				)
+				(hide yes)
 			)
 		)
@@
 					(size 1.27 1.27)
 				)
+				(hide yes)
 			)
 		)
@@
 		(on_board yes)
 		(dnp no)
-		(fields_autoplaced yes)
 		(property "Reference" "R31"
 			(at 58.42 151.1299 0)
@@
 		)
 		(property "Manufacturer_Part_Number" "CRCW08051K00FKEA"
-			(at 60.96 152.4 0)
+			(at 67.564 161.036 0)
 			(effects
 				(font
 					(size 1.27 1.27)
 				)
+				(hide yes)
 			)
 		)
@@
 		)
 		(property "Manufacturer_Part_Number" "2DC2412R-7"
-			(at 58.42 163.83 0)
+			(at 69.088 167.386 0)
 			(effects
 				(font
@@
 					(size 1.27 1.27)
 				)
+				(hide yes)
 			)
 		)
@@
 					(size 1.27 1.27)
 				)
+				(hide yes)
 			)
 		)
@@
 					(size 1.27 1.27)
 				)
+				(hide yes)
 			)
 		)
@@
 					(size 1.27 1.27)
 				)
+				(hide yes)
 			)
 		)
@@
 	(symbol
 		(lib_id "power:GND")
-		(at 101.6 160.02 0)
+		(at 99.06 160.02 0)
 		(mirror y)
 		(unit 1)
@@
 		(dnp no)
 		(property "Reference" "#PWR021"
-			(at 101.6 166.37 0)
+			(at 99.06 166.37 0)
 			(effects
 				(font
@@
 		)
 		(property "Value" "GND"
-			(at 105.156 161.036 0)
+			(at 102.616 161.036 0)
 			(effects
 				(font
@@
 		)
 		(property "Footprint" ""
-			(at 101.6 160.02 0)
+			(at 99.06 160.02 0)
 			(effects
 				(font
@@
 		)
 		(property "Datasheet" ""
-			(at 101.6 160.02 0)
+			(at 99.06 160.02 0)
 			(effects
 				(font
@@
 		)
 		(property "Description" "Power symbol creates a global label with name \"GND\" , ground"
-			(at 101.6 160.02 0)
+			(at 99.06 160.02 0)
 			(effects
 				(font
@@
 			)
 		)
-		(property "Footprint" "MSOP8_MC_MCH"
+		(property "Footprint" "Modelec:MSOP8_MC_MCH"
 			(at 240.03 35.56 0)
 			(effects
@@
 					(size 1.27 1.27)
 				)
+				(hide yes)
 			)
 		)
@@
 					(size 1.27 1.27)
 				)
+				(hide yes)
 			)
 		)
@@
 					(size 1.27 1.27)
 				)
+				(hide yes)
 			)
 		)
@@
 					(size 1.27 1.27)
 				)
+				(hide yes)
 			)
 		)
@@
 					(size 1.27 1.27)
 				)
+				(hide yes)
 			)
 		)
@@
 		(on_board yes)
 		(dnp no)
-		(fields_autoplaced yes)
 		(property "Reference" "J8"
 			(at 35.56 76.1999 0)
@@
 		)
 		(property "Manufacturer_Part_Number" "3220-14-0100-00"
-			(at 46.99 77.47 0)
+			(at 30.226 82.804 0)
 			(effects
 				(font
 					(size 1.27 1.27)
 				)
+				(hide yes)
 			)
 		)
@@
 		(on_board yes)
 		(dnp no)
-		(fields_autoplaced yes)
 		(property "Reference" "BZ1"
 			(at 72.39 151.1299 0)
@@
 		)
 		(property "Manufacturer_Part_Number" "PS1240P02BT"
-			(at 68.58 152.4 0)
+			(at 77.47 156.464 0)
 			(effects
 				(font
@@
 					(size 1.27 1.27)
 				)
+				(hide yes)
 			)
 		)
