File: pcb_puissance/pcb_puissance_2025.kicad_sch (KiCad schematic)
At the start: 20 parts, among them J1 1755736, J2 1755736, J3 1755736, J4 1755736, J5 1755736, J6 1755736

Commit message: dernieres retouches suite changement de repo
Parts:
- PS1: footprint TMR60510 -> Modelec:TMR60510
Changed lines of the file:
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@@
 	(title_block
 		(title "2025 Power supply PCB")
-		(date "2025-02-10")
-		(rev "3")
+		(date "2025-03-06")
+		(rev "4")
 		(company "Modelec")
 		(comment 1 "only 5V, 12V and 24V. Has status leds and communicate status messages via UART.")
@@
 		)
 		(property "Manufacturer_Part_Number" "3568"
-			(at 57.15 48.26 0)
+			(at 62.738 46.736 90)
 			(effects
 				(font
@@
 		)
 		(property "Manufacturer_Part_Number" "3568"
-			(at 57.15 69.85 0)
+			(at 63.5 71.882 90)
 			(effects
 				(font
@@
 		(on_board yes)
 		(dnp no)
-		(fields_autoplaced yes)
 		(property "Reference" "R3"
 			(at 105.41 146.0499 0)
@@
 		)
 		(property "Manufacturer_Part_Number" "CRCW080510K0FKEA"
-			(at 102.87 147.32 0)
+			(at 113.03 141.986 0)
 			(effects
 				(font
 					(size 1.27 1.27)
 				)
+				(hide yes)
 			)
 		)
@@
 			)
 		)
-		(property "Footprint" "TMR60510"
+		(property "Footprint" "Modelec:TMR60510"
 			(at 52.4 176.53 0)
 			(effects
@@
 		)
 		(property "Manufacturer_Part_Number" "3568"
-			(at 57.15 29.21 0)
+			(at 62.738 30.988 90)
 			(effects
 				(font
@@
 		)
 		(property "Manufacturer_Part_Number" "01550900M"
-			(at 144.78 135.89 0)
+			(at 151.892 135.89 0)
 			(effects
 				(font
@@
 		)
 		(property "Sheetname" "power_input_selector"
-			(at 76.2 25.9584 0)
+			(at 76.2 23.1644 0)
 			(effects
 				(font
@@
 		)
 		(property "Sheetfile" "power_input_selector.kicad_sch"
-			(at 76.454 27.94 0)
+			(at 76.2 24.13 0)
 			(effects
 				(font
