File: pcb_puissance/pcb_puissance_2025.kicad_pcb (KiCad board)
At the start: 4 copper layers, 150 x 90 mm, 150 parts, among them J1 1755736, J10 1755736, J11 USB_C_Receptacle_USB2.0_16P, J12 1755736, J13 1755736, J14 Conn_02x06_Odd_Even, J15 1755736, J16 1755736, J17 Conn_02x06_Odd_Even, J18 1755736, J19 1755736, J2 1755736, J20 Conn_02x06_Odd_Even, J21 1755736, J22 1755736, J3 1755736, J4 1755736, J5 1755736, J6 1755736, J7 Conn_02x10_Odd_Even, J8 Conn_ST_STDC14, Q1 SUD50P06-15, Q10 NMOS, Q11 NMOS, Q2 SUD50P06-15, Q3 SUD50P06-15, Q4 SUD50P06-15, Q5 SUD50P06-15, Q6 SUD50P06-15, Q7 STL40DN3LLH5, Q8 NPN, Q9 NMOS, U1 LTC4417IGN, U10 MCP9808T-E/MS, U2 STM32G491KEU6, U3 INA236BIDDFR, U4 INA236AIDDFR, U5 INA236AIDDFR, U6 INA236AIDDFR, U7 INA236BIDDFR, U8 INA236BIDDFR, U9 TCPP02-M18

Commit message: plein de choses que j'avais pas sauvegardé
Connections:
- J8 pad 3: unconnected-(J8-VCC-Pad3) -> /3V3
